File: SensorRadio.sch (KiCad schematic (older format))
At the start: 5 parts, among them P1 ANT, U10 RFM69W, U9 NRF24L01

Commit message: Updated schematics, including w5100
Parts:
- C6, C7: footprint Capacitors_SMD:C_0603_HandSoldering -> Capacitors_SMD:C_0603
Changed lines of the file:
@@
 LIBS:mysensors_arduino
 LIBS:mysensors_logic
+LIBS:mysensors_network
 LIBS:MysensorsGW-cache
 EELAYER 25 0
@@
 $EndComp
 $Comp
-L +3.3V #PWR030
+L +3.3V #PWR033
 U 1 1 553D4655
 P 4350 4350
-F 0 "#PWR030" H 4350 4200 50  0001 C CNN
+F 0 "#PWR033" H 4350 4200 50  0001 C CNN
 F 1 "+3.3V" H 4350 4490 50  0000 C CNN
 F 2 "" H 4350 4350 60  0000 C CNN
@@
 $EndComp
 $Comp
-L +3.3V #PWR031
+L +3.3V #PWR034
 U 1 1 553D4677
 P 4300 2250
-F 0 "#PWR031" H 4300 2100 50  0001 C CNN
+F 0 "#PWR034" H 4300 2100 50  0001 C CNN
 F 1 "+3.3V" H 4300 2390 50  0000 C CNN
 F 2 "" H 4300 2250 60  0000 C CNN
@@
 	4300 2450 4300 2250
 $Comp
-L GND #PWR032
+L GND #PWR035
 U 1 1 553D46D8
 P 4350 5450
-F 0 "#PWR032" H 4350 5200 50  0001 C CNN
+F 0 "#PWR035" H 4350 5200 50  0001 C CNN
 F 1 "GND" H 4350 5300 50  0000 C CNN
 F 2 "" H 4350 5450 60  0000 C CNN
@@
 $EndComp
 $Comp
-L GND #PWR033
+L GND #PWR036
 U 1 1 553D46EE
 P 4250 3600
-F 0 "#PWR033" H 4250 3350 50  0001 C CNN
+F 0 "#PWR036" H 4250 3350 50  0001 C CNN
 F 1 "GND" H 4250 3450 50  0000 C CNN
 F 2 "" H 4250 3600 60  0000 C CNN
@@
 F 0 "C7" H 4625 4500 50  0000 L CNN
 F 1 "C" H 4625 4300 50  0000 L CNN
-F 2 "Capacitors_SMD:C_0603_HandSoldering" H 4638 4250 30  0001 C CNN
+F 2 "Capacitors_SMD:C_0603" H 4638 4250 30  0001 C CNN
 F 3 "" H 4600 4400 60  0000 C CNN
 	1    4600 4400
@@
 F 0 "C6" H 4575 2400 50  0000 L CNN
 F 1 "C" H 4575 2200 50  0000 L CNN
-F 2 "Capacitors_SMD:C_0603_HandSoldering" H 4588 2150 30  0001 C CNN
+F 2 "Capacitors_SMD:C_0603" H 4588 2150 30  0001 C CNN
 F 3 "" H 4550 2300 60  0000 C CNN
 	1    4550 2300
@@
 Connection ~ 4300 2300
 $Comp
-L GND #PWR034
+L GND #PWR037
 U 1 1 553D47FA
 P 4800 2350
-F 0 "#PWR034" H 4800 2100 50  0001 C CNN
+F 0 "#PWR037" H 4800 2100 50  0001 C CNN
 F 1 "GND" H 4800 2200 50  0000 C CNN
 F 2 "" H 4800 2350 60  0000 C CNN
@@
 Connection ~ 3350 4250
 $Comp
-L GND #PWR035
+L GND #PWR038
 U 1 1 553D4A17
 P 4800 4500
-F 0 "#PWR035" H 4800 4250 50  0001 C CNN
+F 0 "#PWR038" H 4800 4250 50  0001 C CNN
 F 1 "GND" H 4800 4350 50  0000 C CNN
 F 2 "" H 4800 4500 60  0000 C CNN
